File: WRTnodeShield/ATMEGA32U4.sch (KiCad schematic (older format))
At the start: 17 parts, among them IC1 IC_ATMEGA32U4_TQFP44, X2 16m

Commit message: 布线完成一部分
Changed lines of the file:
@@
-EESchema Schematic File Version 2  date 2014/11/20 17:18:07
+EESchema Schematic File Version 2  date 2014/11/21 12:19:35
 LIBS:C
 LIBS:IC
@@
 Sheet 3 3
 Title ""
-Date "20 nov 2014"
+Date "21 nov 2014"
 Rev ""
 Comp ""
@@
 U 1 1 545708A7
 P 4750 2950
-F 0 "R21" H 4750 3030 50  0000 C CNN
-F 1 "1M" H 4750 3100 50  0000 C CNN
+F 0 "R21" H 4850 2850 50  0000 C CNN
+F 1 "1M" H 4700 2850 50  0000 C CNN
 F 2 "C_R_0603" H 4750 2830 60  0001 C CNN
 F 3 "~" H 4750 2950 60  0000 C CNN
@@
 U 1 1 54571719
 P 4500 2950
-F 0 "X2" H 4425 3205 50  0000 L BNN
-F 1 "16m" H 4225 2675 50  0000 L BNN
+F 0 "X2" V 4600 3050 50  0000 L BNN
+F 1 "16m" V 4650 2750 50  0000 L BNN
 F 2 "C_CRY_3.2-2.5" H 4500 2600 50  0001 C CNN
 F 3 "~" H 4500 2950 60  0000 C CNN
@@
 U 1 1 54571734
 P 4150 2750
-F 0 "C35" H 4210 2765 50  0000 L BNN
-F 1 "22p" H 3980 2575 50  0000 L BNN
+F 0 "C35" V 4300 2750 50  0000 L BNN
+F 1 "22p" V 4300 2550 50  0000 L BNN
 F 2 "C_C_0603" H 4150 2500 50  0001 C CNN
 F 3 "~" H 4150 2750 60  0000 C CNN
@@
 U 1 1 54571753
 P 4150 3150
-F 0 "C43" H 4210 3165 50  0000 L BNN
-F 1 "22p" H 3980 2975 50  0000 L BNN
+F 0 "C43" V 4250 3150 50  0000 L BNN
+F 1 "22p" V 4100 3150 50  0000 L BNN
 F 2 "C_C_0603" H 4150 2900 50  0001 C CNN
 F 3 "~" H 4150 3150 60  0000 C CNN
@@
 P 1300 2650
 F 0 "C5" H 1360 2665 50  0000 L BNN
-F 1 "100N" H 1130 2475 50  0000 L BNN
+F 1 "100N" H 1350 2500 50  0000 L BNN
 F 2 "C_C_0603" H 1300 2400 50  0001 C CNN
 F 3 "~" H 1300 2650 60  0000 C CNN
@@
 U 1 1 5457187D
 P 1650 2650
-F 0 "C27" H 1710 2665 50  0000 L BNN
-F 1 "100N" H 1480 2475 50  0000 L BNN
+F 0 "C27" H 1500 2700 50  0000 L BNN
+F 1 "100N" H 1450 2500 50  0000 L BNN
 F 2 "C_C_0603" H 1650 2400 50  0001 C CNN
 F 3 "~" H 1650 2650 60  0000 C CNN
@@
 U 1 1 5457192D
 P 1350 3400
-F 0 "L10" V 1256 3250 50  0000 L BNN
+F 0 "L10" V 1500 3350 50  0000 L BNN
 F 1 "L-EUL0603" V 1445 3250 50  0001 L BNN
 F 2 "rcl-L0603" H 1350 3550 50  0001 C CNN
@@
 U 1 1 545719AE
 P 1400 3650
-F 0 "C11" H 1460 3665 50  0000 L BNN
-F 1 "1Uf" H 1230 3475 50  0000 L BNN
+F 0 "C11" V 1500 3650 50  0000 L BNN
+F 1 "1Uf" V 1500 3400 50  0000 L BNN
 F 2 "C_C_0603" H 1400 3400 50  0001 C CNN
 F 3 "~" H 1400 3650 60  0000 C CNN
@@
 P 3200 4300
 F 0 "C29" H 3260 4315 50  0000 L BNN
-F 1 "100N" H 3030 4125 50  0000 L BNN
+F 1 "100N" H 3250 4150 50  0000 L BNN
 F 2 "C_C_0603" H 3200 4050 50  0001 C CNN
 F 3 "~" H 3200 4300 60  0000 C CNN
@@
 U 1 1 5457248F
 P 4600 4200
-F 0 "C44" H 4660 4215 50  0000 L BNN
-F 1 "1Uf" H 4430 4025 50  0000 L BNN
+F 0 "C44" V 4500 4000 50  0000 L BNN
+F 1 "1Uf" V 4750 4000 50  0000 L BNN
 F 2 "C_C_0603" H 4600 3950 50  0001 C CNN
 F 3 "~" H 4600 4200 60  0000 C CNN
@@
 U 1 1 54572856
 P 3600 2050
-F 0 "D1" H 3650 2150 50  0000 L BNN
+F 0 "D1" H 3550 2150 50  0000 L BNN
 F 1 "C_DIODE-1N4148_MINIMELF" H 3100 1809 50  0001 L BNN
 F 2 "C_DIODE-1N4148_MINIMELF" H 3600 2200 50  0001 C CNN
