File: WRTnodeShield/MT7620N.kicad_pcb (KiCad board)
At the start: 2 copper layers, 48 x 45.8 mm, 115 parts, among them IC1 IC_ATMEGA32U4_TQFP44, J1 IO_USB-MICRO-B-MK5P, P2 IO_HOLE-3.2, P3 IO_HOLE-3.2, P3 PINHOLE, Q1 AO3416, Q2 AO3416, T1 AO3415, U1 IC_MP1484EN_SOIC08, U10 DLW21SN900SQ2, U13 IP4220CZ6, U14 IP4220CZ6, U15 AP2146, U16 AP2146, U2 DLW21SN900SQ2, U3 IP4220CZ6, U4 UPD720114-QFP48, U5 USB-AF-90, U9 DLW21SN900SQ2, X1 30MHz, X2 16m

Commit message: 布线完成一部分
Parts:
- removed the P3 at (129.9, 59.4)
- J1: moved to F.Cu
- moved C6 3.56 mm to (165.8, 61.8)
- moved C23 2.03 mm to (165.8, 63.6)
- moved C24 1.91 mm to (165.8, 65.4)
- moved J1 0.26 mm to (205.7, 64.0), turned to 90 degrees
- moved C12 0.05 mm to (165.8, 71.1)
- moved R10 0.05 mm to (165.8, 67.3)
- moved R9 0.05 mm to (165.8, 69.2)
- turned C9 to 180 degrees
- turned L10 to 0 degrees
- turned R23 to 0 degrees
Routing:
- net GND: track 1.91 -> 58.5 mm
- net /uPD720114/HUB33V: track 0.00 -> 55.7 mm
- net +5V: track 0.00 -> 46.7 mm
- net N-00000112: track 0.00 -> 39.2 mm
- net +3.3V: track 0.00 -> 34.3 mm
- net /ATMEGA32U4/D6*: track 0.00 -> 33.7 mm
- net /uPD720114/VBUS1: track 0.00 -> 31.4 mm, vias 0 -> 2
- net /ATMEGA32U4/IO8: track 0.00 -> 28.7 mm, vias 0 -> 1
- net /ATMEGA32U4/IO9*: track 0.00 -> 27.9 mm, vias 0 -> 1
- net N-0000024: track 0.00 -> 26.2 mm
- net /ATMEGA32U4/IO12: track 0.00 -> 24.8 mm
- net /uPD720114/VBUS2: track 0.00 -> 22.7 mm, vias 0 -> 2
- net N-00000113: track 0.00 -> 20.1 mm
- net N-0000081: track 9.25 -> 28.2 mm, vias 0 -> 2
- net N-00000107: track 0.00 -> 18.3 mm
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- added copper zone on F.Cu, net +3.3V
- added copper zone on F.Cu, net +5V
- added copper zone on F.Cu, net GND
- added copper zone on F.Cu, net N-000001
- added copper zone on F.Cu, net N-0000022
