File: WRTnodeShield/uPD720114.sch (KiCad schematic (older format))
At the start: 60 parts, among them U10 DLW21SN900SQ2, U13 IP4220CZ6, U14 IP4220CZ6, U15 AP2146, U16 AP2146, U2 DLW21SN900SQ2, U3 IP4220CZ6, U4 UPD720114-QFP48, U5 USB-AF-90, U9 DLW21SN900SQ2, X1 30MHz

Commit message: 布线完成一部分
Changed lines of the file:
@@
-EESchema Schematic File Version 2  date 2014/11/20 17:18:07
+EESchema Schematic File Version 2  date 2014/11/21 12:19:35
 LIBS:C
 LIBS:IC
@@
 Sheet 2 3
 Title ""
-Date "20 nov 2014"
+Date "21 nov 2014"
 Rev ""
 Comp ""
@@
 U 1 1 534FC3D3
 P 8500 5450
-F 0 "C28" H 8560 5465 50  0000 L BNN
-F 1 "0.1uF" H 8330 5275 50  0000 L BNN
+F 0 "C28" H 8350 5450 50  0000 L BNN
+F 1 "0.1uF" H 8300 5250 50  0000 L BNN
 F 2 "C_C_0603" H 8500 5200 50  0001 C CNN
 F 3 "~" H 8500 5450 60  0000 C CNN
@@
 U 1 1 534FC3E5
 P 8600 6450
-F 0 "C30" H 8660 6465 50  0000 L BNN
-F 1 "0.1uF" H 8430 6275 50  0000 L BNN
+F 0 "C30" H 8450 6500 50  0000 L BNN
+F 1 "0.1uF" H 8600 6250 50  0000 L BNN
 F 2 "C_C_0603" H 8600 6200 50  0001 C CNN
 F 3 "~" H 8600 6450 60  0000 C CNN
@@
 U 1 1 5369D496
 P 9000 5350
-F 0 "C31" H 9095 5419 50  0000 L BNN
-F 1 "68uF" H 9095 5309 50  0000 L BNN
+F 0 "C31" H 8800 5400 50  0000 L BNN
+F 1 "68uF" H 8800 5250 50  0000 L BNN
 F 2 "C_CPOL_SMCB" H 9020 5130 50  0001 C CNN
 F 3 "~" H 9000 5350 60  0000 C CNN
@@
 U 1 1 5369D4CC
 P 9400 5350
-F 0 "C33" H 9495 5419 50  0000 L BNN
-F 1 "68uF" H 9495 5309 50  0000 L BNN
+F 0 "C33" H 9250 5450 50  0000 L BNN
+F 1 "68uF" H 9250 5250 50  0000 L BNN
 F 2 "C_CPOL_SMCB" H 9420 5130 50  0001 C CNN
 F 3 "~" H 9400 5350 60  0000 C CNN
@@
 U 1 1 5369D4DE
 P 9000 6500
-F 0 "C32" H 9095 6569 50  0000 L BNN
-F 1 "68uF" H 9095 6459 50  0000 L BNN
+F 0 "C32" H 8850 6600 50  0000 L BNN
+F 1 "68uF" H 9000 6350 50  0000 L BNN
 F 2 "C_CPOL_SMCB" H 9020 6280 50  0001 C CNN
 F 3 "~" H 9000 6500 60  0000 C CNN
@@
 U 1 1 5369D4F0
 P 9400 6500
-F 0 "C34" H 9495 6569 50  0000 L BNN
-F 1 "68uF" H 9495 6459 50  0000 L BNN
+F 0 "C34" H 9250 6600 50  0000 L BNN
+F 1 "68uF" H 9400 6350 50  0000 L BNN
 F 2 "C_CPOL_SMCB" H 9420 6280 50  0001 C CNN
 F 3 "~" H 9400 6500 60  0000 C CNN
@@
 U 1 1 5369D506
 P 8700 5500
-F 0 "C37" H 8795 5569 50  0000 L BNN
-F 1 "10uF" H 8795 5459 50  0000 L BNN
+F 0 "C37" H 8550 5600 50  0000 L BNN
+F 1 "10uF" H 8500 5350 50  0000 L BNN
 F 2 "C_CPOL_SMCA" H 8720 5280 50  0001 C CNN
 F 3 "~" H 8700 5500 60  0000 C CNN
@@
 U 1 1 5369D7CA
 P 8800 6500
-F 0 "C38" H 8895 6569 50  0000 L BNN
-F 1 "10uF" H 8895 6459 50  0000 L BNN
+F 0 "C38" H 8650 6600 50  0000 L BNN
+F 1 "10uF" H 8800 6350 50  0000 L BNN
 F 2 "C_CPOL_SMCA" H 8820 6280 50  0001 C CNN
 F 3 "~" H 8800 6500 60  0000 C CNN
@@
 U 1 1 5369DA97
 P 9200 5300
-F 0 "C39" H 9260 5315 50  0000 L BNN
+F 0 "C39" H 9050 5300 50  0000 L BNN
 F 1 "0.1uF" H 9030 5125 50  0000 L BNN
 F 2 "C_C_0603" H 9200 5050 50  0001 C CNN
@@
 P 9600 5300
 F 0 "C41" H 9660 5315 50  0000 L BNN
-F 1 "0.1uF" H 9430 5125 50  0000 L BNN
+F 1 "0.1uF" H 9650 5150 50  0000 L BNN
 F 2 "C_C_0603" H 9600 5050 50  0001 C CNN
 F 3 "~" H 9600 5300 60  0000 C CNN
@@
 U 1 1 5369DAA3
 P 9200 6450
-F 0 "C40" H 9260 6465 50  0000 L BNN
-F 1 "0.1uF" H 9030 6275 50  0000 L BNN
+F 0 "C40" H 9050 6500 50  0000 L BNN
+F 1 "0.1uF" H 9200 6250 50  0000 L BNN
 F 2 "C_C_0603" H 9200 6200 50  0001 C CNN
 F 3 "~" H 9200 6450 60  0000 C CNN
@@
 U 1 1 5369DAA9
 P 9650 6450
-F 0 "C42" H 9710 6465 50  0000 L BNN
-F 1 "0.1uF" H 9480 6275 50  0000 L BNN
+F 0 "C42" H 9500 6500 50  0000 L BNN
+F 1 "0.1uF" H 9650 6250 50  0000 L BNN
 F 2 "C_C_0603" H 9650 6200 50  0001 C CNN
 F 3 "~" H 9650 6450 60  0000 C CNN
@@
 U 1 1 54575999
 P 9800 3100
-F 0 "U5" H 9800 3550 60  0000 C CNN
-F 1 "USB-AF-90" H 9800 3650 60  0000 C CNN
+F 0 "U5" H 9700 3400 60  0000 C CNN
+F 1 "USB-AF-90" H 9750 3500 60  0000 C CNN
 F 2 "USB-AF-90" H 9800 3100 60  0001 C CNN
 F 3 "~" H 9800 3100 60  0000 C CNN
