File: ATMEGA32U4.sch (KiCad schematic (older format))
At the start: 17 parts, among them IC1 IC_ATMEGA32U4_TQFP44, X2 16m

Commit message: 整理到根目录
Parts:
- added JP11: IO_M02X1, IO_M02X1, symbol IO_M02X1
Connections:
- net +5V: now also JP11.1
- net D5*: now also JP4.10; no longer JP4.5
- net D7: now also JP4.12; no longer JP4.7
- net GND: now also JP11.2
- net IO10*: now also JP4.9; no longer JP4.10
- net IO11*: now also JP4.13; no longer JP4.11
- net IO12: now also JP4.5; no longer JP4.12
- net IO13*: now also JP4.11; no longer JP4.13
- net IO8: now also JP4.7; no longer JP4.8
- net IO9*: now also JP4.8; no longer JP4.9
Changed lines of the file:
@@
-EESchema Schematic File Version 2  date 2014/11/21 12:19:35
+EESchema Schematic File Version 2  date 2014/11/26 13:45:51
 LIBS:C
 LIBS:IC
@@
 Sheet 3 3
 Title ""
-Date "21 nov 2014"
+Date "26 nov 2014"
 Rev ""
 Comp ""
@@
 $EndComp
 $Comp
-L GND #PWR049
+L GND #PWR050
 U 1 1 545717EF
 P 3950 3450
-F 0 "#PWR049" H 3950 3450 30  0001 C CNN
+F 0 "#PWR050" H 3950 3450 30  0001 C CNN
 F 1 "GND" H 3950 3380 30  0001 C CNN
 F 2 "" H 3950 3450 60  0000 C CNN
@@
 $EndComp
 $Comp
-L AGND #PWR050
+L AGND #PWR051
 U 1 1 54571814
 P 4550 2500
-F 0 "#PWR050" H 4550 2500 40  0001 C CNN
+F 0 "#PWR051" H 4550 2500 40  0001 C CNN
 F 1 "AGND" H 4550 2430 50  0000 C CNN
 F 2 "" H 4550 2500 60  0000 C CNN
@@
 MCU5V
 $Comp
-L GND #PWR051
+L GND #PWR052
 U 1 1 545718DD
 P 1450 3000
-F 0 "#PWR051" H 1450 3000 30  0001 C CNN
+F 0 "#PWR052" H 1450 3000 30  0001 C CNN
 F 1 "GND" H 1450 2930 30  0001 C CNN
 F 2 "" H 1450 3000 60  0000 C CNN
@@
 $EndComp
 $Comp
-L GND #PWR052
+L GND #PWR053
 U 1 1 545719E9
 P 1000 3850
-F 0 "#PWR052" H 1000 3850 30  0001 C CNN
+F 0 "#PWR053" H 1000 3850 30  0001 C CNN
 F 1 "GND" H 1000 3780 30  0001 C CNN
 F 2 "" H 1000 3850 60  0000 C CNN
@@
 AREF
 $Comp
-L AGND #PWR053
+L AGND #PWR054
 U 1 1 54571ED3
 P 3200 4950
-F 0 "#PWR053" H 3200 4950 40  0001 C CNN
+F 0 "#PWR054" H 3200 4950 40  0001 C CNN
 F 1 "AGND" H 3200 4880 50  0000 C CNN
 F 2 "" H 3200 4950 60  0000 C CNN
@@
 MCU5V
 $Comp
-L GND #PWR054
+L GND #PWR055
 U 1 1 54572002
 P 4650 4050
-F 0 "#PWR054" H 4650 4050 30  0001 C CNN
+F 0 "#PWR055" H 4650 4050 30  0001 C CNN
 F 1 "GND" H 4650 3980 30  0001 C CNN
 F 2 "" H 4650 4050 60  0000 C CNN
@@
 $EndComp
 $Comp
-L GND #PWR055
+L GND #PWR056
 U 1 1 54572605
 P 3800 4950
-F 0 "#PWR055" H 3800 4950 30  0001 C CNN
+F 0 "#PWR056" H 3800 4950 30  0001 C CNN
 F 1 "GND" H 3800 4880 30  0001 C CNN
 F 2 "" H 3800 4950 60  0000 C CNN
@@
 UGND
 $Comp
-L GND #PWR056
+L GND #PWR057
 U 1 1 54572760
 P 4750 5550
-F 0 "#PWR056" H 4750 5550 30  0001 C CNN
+F 0 "#PWR057" H 4750 5550 30  0001 C CNN
 F 1 "GND" H 4750 5480 30  0001 C CNN
 F 2 "" H 4750 5550 60  0000 C CNN
@@
 $EndComp
 $Comp
-L GND #PWR057
+L GND #PWR058
 U 1 1 54572805
 P 7350 4650
-F 0 "#PWR057" H 7350 4650 30  0001 C CNN
+F 0 "#PWR058" H 7350 4650 30  0001 C CNN
 F 1 "GND" H 7350 4580 30  0001 C CNN
 F 2 "" H 7350 4650 60  0000 C CNN
@@
 Wire Wire Line
 	6700 2400 6950 2400
-Text Label 8450 2900 0    60   ~ 0
+Text Label 8450 3000 0    60   ~ 0
 IO11*
 Text Label 10100 2500 0    60   ~ 0
@@
 Text Label 10100 2400 0    60   ~ 0
 D1/TX
-Text Label 10100 2900 0    60   ~ 0
+Text Label 8450 2600 0    60   ~ 0
 IO12
 Text Label 10100 2600 0    60   ~ 0
 D6*
+Text Label 8450 2700 0    60   ~ 0
+IO8
 Text Label 10100 2700 0    60   ~ 0
-IO8
+IO9*
 Text Label 8450 2800 0    60   ~ 0
-IO9*
+IO10*
 Text Label 10100 2800 0    60   ~ 0
-IO10*
-Text Label 8450 2600 0    60   ~ 0
 D5*
-Text Label 8450 3000 0    60   ~ 0
+Text Label 8450 2900 0    60   ~ 0
 IO13*
 Text Label 10100 3000 0    60   ~ 0
@@
 Text Label 8450 3300 0    60   ~ 0
 A5
-Text Label 8450 2700 0    60   ~ 0
+Text Label 10100 2900 0    60   ~ 0
 D7
 Wire Wire Line
@@
 	8850 3500 8450 3500
 $Comp
-L +5V #PWR058
+L +5V #PWR059
 U 1 1 546E00A5
 P 10100 3400
-F 0 "#PWR058" H 10100 3490 20  0001 C CNN
+F 0 "#PWR059" H 10100 3490 20  0001 C CNN
 F 1 "+5V" H 10100 3490 30  0000 C CNN
 F 2 "" H 10100 3400 60  0000 C CNN
@@
 $EndComp
 $Comp
-L GND #PWR059
+L GND #PWR060
 U 1 1 546E00BF
 P 10100 3700
-F 0 "#PWR059" H 10100 3700 30  0001 C CNN
+F 0 "#PWR060" H 10100 3700 30  0001 C CNN
 F 1 "GND" H 10100 3630 30  0001 C CNN
 F 2 "" H 10100 3700 60  0000 C CNN
@@
 	10100 3600 10100 3700
 $Comp
-L +5V #PWR060
+L +5V #PWR061
 U 1 1 546E13FD
 P 10100 3300
-F 0 "#PWR060" H 10100 3390 20  0001 C CNN
+F 0 "#PWR061" H 10100 3390 20  0001 C CNN
 F 1 "+5V" H 10100 3390 30  0000 C CNN
 F 2 "" H 10100 3300 60  0000 C CNN
@@
 	0    1    1    0
 $EndComp
+$Comp
+L IO_M02X1 JP11
+U 1 1 54744238
+P 9300 4350
+F 0 "JP11" H 9280 4160 60  0000 C CNN
+F 1 "IO_M02X1" H 9290 4540 60  0000 C CNN
+F 2 "IO_M02X1" H 9290 4540 60  0001 C CNN
+F 3 "~" H 9300 4350 60  0000 C CNN
+	1    9300 4350
+	1    0    0    -1
+$EndComp
+$Comp
+L +5V #PWR062
+U 1 1 54744245
+P 9700 4300
+F 0 "#PWR062" H 9700 4390 20  0001 C CNN
+F 1 "+5V" H 9700 4390 30  0000 C CNN
+F 2 "" H 9700 4300 60  0000 C CNN
+F 3 "" H 9700 4300 60  0000 C CNN
+	1    9700 4300
+	0    1    1    0
+$EndComp
+$Comp
+L GND #PWR063
+U 1 1 5474424B
+P 9700 4500
+F 0 "#PWR063" H 9700 4500 30  0001 C CNN
+F 1 "GND" H 9700 4430 30  0001 C CNN
+F 2 "" H 9700 4500 60  0000 C CNN
+F 3 "" H 9700 4500 60  0000 C CNN
+	1    9700 4500
+	1    0    0    -1
+$EndComp
+Wire Wire Line
+	9550 4300 9700 4300
+Wire Wire Line
+	9550 4400 9700 4400
+Wire Wire Line
+	9700 4400 9700 4500
 $EndSCHEMATC

Commit message: 生成gerber文件并整理目录
Connections:
- net +5V: no longer JP4.20
- net AREF: now also JP4.20
Changed lines of the file:
@@
-EESchema Schematic File Version 2  date 2014/11/26 13:45:51
-LIBS:C
-LIBS:IC
+EESchema Schematic File Version 2  date 2014/11/27 13:40:31
 LIBS:power
-LIBS:rcl
-LIBS:gl
-LIBS:I-O
-LIBS:REQUEST
-LIBS:SchumyHao
+LIBS:5V DC ADAPTER-cache
+LIBS:5V to 3.3V-cache
+LIBS:ATMEGA32U4-cache
 LIBS:MT7620N-cache
+LIBS:uPD720114-cache
+LIBS:WLAN-cache
 EELAYER 27 0
 EELAYER END
@@
 Sheet 3 3
 Title ""
-Date "26 nov 2014"
+Date "27 nov 2014"
 Rev ""
 Comp ""
@@
 $EndComp
 $Comp
-L GND #PWR050
+L GND #PWR54
 U 1 1 545717EF
 P 3950 3450
-F 0 "#PWR050" H 3950 3450 30  0001 C CNN
+F 0 "#PWR54" H 3950 3450 30  0001 C CNN
 F 1 "GND" H 3950 3380 30  0001 C CNN
 F 2 "" H 3950 3450 60  0000 C CNN
@@
 $EndComp
 $Comp
-L AGND #PWR051
+L AGND #PWR55
 U 1 1 54571814
 P 4550 2500
-F 0 "#PWR051" H 4550 2500 40  0001 C CNN
+F 0 "#PWR55" H 4550 2500 40  0001 C CNN
 F 1 "AGND" H 4550 2430 50  0000 C CNN
 F 2 "" H 4550 2500 60  0000 C CNN
@@
 MCU5V
 $Comp
-L GND #PWR052
+L GND #PWR51
 U 1 1 545718DD
 P 1450 3000
-F 0 "#PWR052" H 1450 3000 30  0001 C CNN
+F 0 "#PWR51" H 1450 3000 30  0001 C CNN
 F 1 "GND" H 1450 2930 30  0001 C CNN
 F 2 "" H 1450 3000 60  0000 C CNN
@@
 $EndComp
 $Comp
-L GND #PWR053
+L GND #PWR50
 U 1 1 545719E9
 P 1000 3850
-F 0 "#PWR053" H 1000 3850 30  0001 C CNN
+F 0 "#PWR50" H 1000 3850 30  0001 C CNN
 F 1 "GND" H 1000 3780 30  0001 C CNN
 F 2 "" H 1000 3850 60  0000 C CNN
@@
 AREF
 $Comp
-L AGND #PWR054
+L AGND #PWR52
 U 1 1 54571ED3
 P 3200 4950
-F 0 "#PWR054" H 3200 4950 40  0001 C CNN
+F 0 "#PWR52" H 3200 4950 40  0001 C CNN
 F 1 "AGND" H 3200 4880 50  0000 C CNN
 F 2 "" H 3200 4950 60  0000 C CNN
@@
 MCU5V
 $Comp
-L GND #PWR055
+L GND #PWR56
 U 1 1 54572002
 P 4650 4050
-F 0 "#PWR055" H 4650 4050 30  0001 C CNN
+F 0 "#PWR56" H 4650 4050 30  0001 C CNN
 F 1 "GND" H 4650 3980 30  0001 C CNN
 F 2 "" H 4650 4050 60  0000 C CNN
@@
 $EndComp
 $Comp
-L GND #PWR056
+L GND #PWR53
 U 1 1 54572605
 P 3800 4950
-F 0 "#PWR056" H 3800 4950 30  0001 C CNN
+F 0 "#PWR53" H 3800 4950 30  0001 C CNN
 F 1 "GND" H 3800 4880 30  0001 C CNN
 F 2 "" H 3800 4950 60  0000 C CNN
@@
 UGND
 $Comp
-L GND #PWR057
+L GND #PWR57
 U 1 1 54572760
 P 4750 5550
-F 0 "#PWR057" H 4750 5550 30  0001 C CNN
+F 0 "#PWR57" H 4750 5550 30  0001 C CNN
 F 1 "GND" H 4750 5480 30  0001 C CNN
 F 2 "" H 4750 5550 60  0000 C CNN
@@
 $EndComp
 $Comp
-L GND #PWR058
+L GND #PWR58
 U 1 1 54572805
 P 7350 4650
-F 0 "#PWR058" H 7350 4650 30  0001 C CNN
+F 0 "#PWR58" H 7350 4650 30  0001 C CNN
 F 1 "GND" H 7350 4580 30  0001 C CNN
 F 2 "" H 7350 4650 60  0000 C CNN
@@
 	8850 3500 8450 3500
 $Comp
-L +5V #PWR059
+L +5V #PWR61
 U 1 1 546E00A5
 P 10100 3400
-F 0 "#PWR059" H 10100 3490 20  0001 C CNN
+F 0 "#PWR61" H 10100 3490 20  0001 C CNN
 F 1 "+5V" H 10100 3490 30  0000 C CNN
 F 2 "" H 10100 3400 60  0000 C CNN
@@
 $EndComp
 $Comp
-L GND #PWR060
+L GND #PWR62
 U 1 1 546E00BF
 P 10100 3700
-F 0 "#PWR060" H 10100 3700 30  0001 C CNN
+F 0 "#PWR62" H 10100 3700 30  0001 C CNN
 F 1 "GND" H 10100 3630 30  0001 C CNN
 F 2 "" H 10100 3700 60  0000 C CNN
@@
 	10100 3600 10100 3700
 $Comp
-L +5V #PWR061
-U 1 1 546E13FD
-P 10100 3300
-F 0 "#PWR061" H 10100 3390 20  0001 C CNN
-F 1 "+5V" H 10100 3390 30  0000 C CNN
-F 2 "" H 10100 3300 60  0000 C CNN
-F 3 "" H 10100 3300 60  0000 C CNN
-	1    10100 3300
-	0    1    1    0
-$EndComp
-$Comp
 L IO_M02X1 JP11
 U 1 1 54744238
@@
 $EndComp
 $Comp
-L +5V #PWR062
+L +5V #PWR59
 U 1 1 54744245
 P 9700 4300
-F 0 "#PWR062" H 9700 4390 20  0001 C CNN
+F 0 "#PWR59" H 9700 4390 20  0001 C CNN
 F 1 "+5V" H 9700 4390 30  0000 C CNN
 F 2 "" H 9700 4300 60  0000 C CNN
@@
 $EndComp
 $Comp
-L GND #PWR063
+L GND #PWR60
 U 1 1 5474424B
 P 9700 4500
-F 0 "#PWR063" H 9700 4500 30  0001 C CNN
+F 0 "#PWR60" H 9700 4500 30  0001 C CNN
 F 1 "GND" H 9700 4430 30  0001 C CNN
 F 2 "" H 9700 4500 60  0000 C CNN
@@
 Wire Wire Line
 	9700 4400 9700 4500
+Text Label 10100 3300 0    60   ~ 0
+AREF
 $EndSCHEMATC
