File: MT7620N.sch (KiCad schematic (older format))
At the start: 35 parts, among them J1 IO_USB-MICRO-B-MK5P, P2 IO_HOLE-3.2, P3 IO_HOLE-3.2, Q1 AO3416, Q2 AO3416, T1 AO3415, U1 IC_MP1484EN_SOIC08

Commit message: 整理到根目录
Parts:
- removed JP3: IO_M05X2, IO_M05X2, symbol IO_M05X2
- added JP10, JP3, JP8: IO_M02X1, IO_M02X1, symbol IO_M02X1
Connections:
- net +5V: now also R26.2
- net GND: now also JP3.1
- net I2C_SCLK: now also JP8.1
- net I2C_SD: now also JP8.2
- net LINK3: now also JP10.2
- net LINK4: now also JP10.1
- net MCU5V: no longer R26.2
- net WRT33V: now also JP3.2
Changed lines of the file:
@@
-EESchema Schematic File Version 2  date 2014/11/21 12:19:35
+EESchema Schematic File Version 2  date 2014/11/26 13:45:51
 LIBS:C
 LIBS:IC
@@
 Sheet 1 3
 Title ""
-Date "21 nov 2014"
+Date "26 nov 2014"
 Rev ""
 Comp ""
@@
 	0    -1   -1   0
 $EndComp
-Text Label 2650 6100 2    60   ~ 0
-SPI_MISO
-Text Label 4000 6100 0    60   ~ 0
-SPI_MOSI
-Text Label 2650 6200 2    60   ~ 0
-SPI_WP
-Text Label 4000 6200 0    60   ~ 0
-SPI_HOLD
-Text Label 2650 6300 2    60   ~ 0
-SPI_CLK
-Text Label 4000 6300 0    60   ~ 0
-SPI_CS1
 Text Label 2650 6400 2    60   ~ 0
 I2C_SCLK
@@
 	0    -1   -1   0
 $EndComp
-Text Label 6800 4000 0    60   ~ 0
-MCU5V
 Wire Wire Line
 	6350 4600 7200 4600
@@
 $EndSheet
 Wire Wire Line
-	3750 6100 4000 6100
-Wire Wire Line
-	3750 6200 4000 6200
-Wire Wire Line
-	3750 6300 4000 6300
-Wire Wire Line
-	3750 6400 4000 6400
-Wire Wire Line
-	2650 6100 2850 6100
-Wire Wire Line
-	2650 6200 2850 6200
-Wire Wire Line
-	2650 6300 2850 6300
-Wire Wire Line
-	2650 6400 2850 6400
-$Comp
-L IO_M05X2 JP3
-U 1 1 546DF7F7
-P 3250 6100
-F 0 "JP3" H 3280 6445 60  0000 C CNN
-F 1 "IO_M05X2" H 3300 6350 60  0000 C CNN
-F 2 "IO_M05X2" H 3305 5665 60  0001 C CNN
-F 3 "~" H 3250 6100 60  0000 C CNN
-	1    3250 6100
-	1    0    0    -1
-$EndComp
+	3300 6400 4000 6400
+Wire Wire Line
+	2650 6400 3200 6400
 Text Label 2650 6000 2    60   ~ 0
 WRT33V
 Wire Wire Line
-	3750 6000 4000 6000
-Wire Wire Line
-	2850 6000 2650 6000
+	3300 6000 4000 6000
+Wire Wire Line
+	2650 6000 3200 6000
 $Comp
 L AO3416 Q2
@@
 	1    0    0    -1
 $EndComp
+$Comp
+L IO_M02X1 JP3
+U 1 1 5474263A
+P 3250 5750
+F 0 "JP3" H 3230 5560 60  0000 C CNN
+F 1 "IO_M02X1" H 3240 5940 60  0000 C CNN
+F 2 "IO_M02X1" H 3240 5940 60  0001 C CNN
+F 3 "~" H 3250 5750 60  0000 C CNN
+	1    3250 5750
+	0    1    1    0
+$EndComp
+$Comp
+L IO_M02X1 JP8
+U 1 1 547429BF
+P 3250 6650
+F 0 "JP8" H 3230 6460 60  0000 C CNN
+F 1 "IO_M02X1" H 3240 6840 60  0000 C CNN
+F 2 "IO_M02X1" H 3240 6840 60  0001 C CNN
+F 3 "~" H 3250 6650 60  0000 C CNN
+	1    3250 6650
+	0    -1   -1   0
+$EndComp
+$Comp
+L +5V #PWR019
+U 1 1 54752FD0
+P 6800 4000
+F 0 "#PWR019" H 6800 4090 20  0001 C CNN
+F 1 "+5V" H 6800 4090 30  0000 C CNN
+F 2 "~" H 6800 4000 60  0000 C CNN
+F 3 "~" H 6800 4000 60  0000 C CNN
+	1    6800 4000
+	1    0    0    -1
+$EndComp
+$Comp
+L IO_M02X1 JP10
+U 1 1 54756997
+P 3600 2500
+F 0 "JP10" H 3580 2310 60  0000 C CNN
+F 1 "IO_M02X1" H 3590 2690 60  0000 C CNN
+F 2 "IO_M02X1" H 3590 2690 60  0001 C CNN
+F 3 "~" H 3600 2500 60  0000 C CNN
+	1    3600 2500
+	-1   0    0    1
+$EndComp
+Wire Wire Line
+	3350 2450 3050 2450
+Wire Wire Line
+	3350 2550 3050 2550
+Text Label 3050 2550 0    60   ~ 0
+LINK4
+Text Label 3050 2450 0    60   ~ 0
+LINK3
 $EndSCHEMATC

Commit message: 生成gerber文件并整理目录
Parts:
- added R28: NO, C_R_0603, symbol C_R_0603
Connections:
- net +5V: now also R28.2
- net MCU5V: now also R28.1
Changed lines of the file:
@@
-EESchema Schematic File Version 2  date 2014/11/26 13:45:51
-LIBS:C
-LIBS:IC
+EESchema Schematic File Version 2  date 2014/11/27 13:40:31
 LIBS:power
-LIBS:rcl
-LIBS:gl
-LIBS:I-O
-LIBS:REQUEST
-LIBS:SchumyHao
+LIBS:5V DC ADAPTER-cache
+LIBS:5V to 3.3V-cache
+LIBS:ATMEGA32U4-cache
 LIBS:MT7620N-cache
+LIBS:uPD720114-cache
+LIBS:WLAN-cache
 EELAYER 27 0
 EELAYER END
@@
 Sheet 1 3
 Title ""
-Date "26 nov 2014"
+Date "27 nov 2014"
 Rev ""
 Comp ""
@@
 $EndDescr
 $Comp
-L GND #PWR01
+L GND #PWR3
 U 1 1 5265E21E
 P 2950 1600
-F 0 "#PWR01" H 2950 1600 30  0001 C CNN
+F 0 "#PWR3" H 2950 1600 30  0001 C CNN
 F 1 "GND" H 2950 1530 30  0001 C CNN
 F 2 "" H 2950 1600 60  0000 C CNN
@@
 LINK4
 $Comp
-L GND #PWR02
+L GND #PWR4
 U 1 1 5265EC1D
 P 3000 3250
-F 0 "#PWR02" H 3000 3250 30  0001 C CNN
+F 0 "#PWR4" H 3000 3250 30  0001 C CNN
 F 1 "GND" H 3000 3180 30  0001 C CNN
 F 2 "" H 3000 3250 60  0000 C CNN
@@
 PA_PE_G1
 $Comp
-L GND #PWR03
+L GND #PWR2
 U 1 1 5265F363
 P 850 3150
-F 0 "#PWR03" H 850 3150 30  0001 C CNN
+F 0 "#PWR2" H 850 3150 30  0001 C CNN
 F 1 "GND" H 850 3080 30  0001 C CNN
 F 2 "" H 850 3150 60  0000 C CNN
@@
 D+
 $Comp
-L GND #PWR04
+L GND #PWR1
 U 1 1 52845B01
 P 650 2500
-F 0 "#PWR04" H 650 2400 30  0001 C CNN
+F 0 "#PWR1" H 650 2400 30  0001 C CNN
 F 1 "GND" H 650 2430 30  0001 C CNN
 F 2 "~" H 650 2500 60  0000 C CNN
@@
 $EndComp
 $Comp
-L GND #PWR05
+L GND #PWR9
 U 1 1 52D56EAB
 P 5900 1550
-F 0 "#PWR05" H 5900 1450 30  0001 C CNN
+F 0 "#PWR9" H 5900 1450 30  0001 C CNN
 F 1 "GND" H 5900 1480 30  0001 C CNN
 F 2 "~" H 5900 1550 60  0000 C CNN
@@
 NoConn ~ 4850 1350
 $Comp
-L GND #PWR06
+L GND #PWR7
 U 1 1 52D57199
 P 4900 2050
-F 0 "#PWR06" H 4900 1950 30  0001 C CNN
+F 0 "#PWR7" H 4900 1950 30  0001 C CNN
 F 1 "GND" H 4900 1980 30  0001 C CNN
 F 2 "~" H 4900 2050 60  0000 C CNN
@@
 $EndComp
 $Comp
-L GND #PWR07
+L GND #PWR5
 U 1 1 52D65C33
 P 4000 6000
-F 0 "#PWR07" H 4000 5900 30  0001 C CNN
+F 0 "#PWR5" H 4000 5900 30  0001 C CNN
 F 1 "GND" H 4000 5930 30  0001 C CNN
 F 2 "~" H 4000 6000 60  0000 C CNN
@@
 NoConn ~ 4850 1250
 $Comp
-L +5V #PWR08
+L +5V #PWR10
 U 1 1 534DE5AB
 P 6650 900
-F 0 "#PWR08" H 6650 990 20  0001 C CNN
+F 0 "#PWR10" H 6650 990 20  0001 C CNN
 F 1 "+5V" H 6650 990 30  0000 C CNN
 F 2 "~" H 6650 900 60  0000 C CNN
@@
 $EndComp
 $Comp
-L GND #PWR09
+L GND #PWR11
 U 1 1 534DE5CC
 P 6650 2500
-F 0 "#PWR09" H 6650 2500 30  0001 C CNN
+F 0 "#PWR11" H 6650 2500 30  0001 C CNN
 F 1 "GND" H 6650 2430 30  0001 C CNN
 F 2 "" H 6650 2500 60  0000 C CNN
@@
 $EndComp
 $Comp
-L +3.3V #PWR010
+L +3.3V #PWR16
 U 1 1 534DFBDE
 P 10150 900
-F 0 "#PWR010" H 10150 860 30  0001 C CNN
+F 0 "#PWR16" H 10150 860 30  0001 C CNN
 F 1 "+3.3V" H 10150 1010 30  0000 C CNN
 F 2 "" H 10150 900 60  0000 C CNN
@@
 $EndComp
 $Comp
-L GND #PWR011
+L GND #PWR13
 U 1 1 534DFE0F
 P 7050 2500
-F 0 "#PWR011" H 7050 2500 30  0001 C CNN
+F 0 "#PWR13" H 7050 2500 30  0001 C CNN
 F 1 "GND" H 7050 2430 30  0001 C CNN
 F 2 "" H 7050 2500 60  0000 C CNN
@@
 $EndComp
 $Comp
-L GND #PWR012
+L GND #PWR15
 U 1 1 534E0047
 P 7900 3500
-F 0 "#PWR012" H 7900 3500 30  0001 C CNN
+F 0 "#PWR15" H 7900 3500 30  0001 C CNN
 F 1 "GND" H 7900 3430 30  0001 C CNN
 F 2 "" H 7900 3500 60  0000 C CNN
@@
 $EndComp
 $Comp
-L +3.3V #PWR013
+L +3.3V #PWR17
 U 1 1 53670B5B
 P 10600 900
-F 0 "#PWR013" H 10600 860 30  0001 C CNN
+F 0 "#PWR17" H 10600 860 30  0001 C CNN
 F 1 "+3.3V" H 10600 1010 30  0000 C CNN
 F 2 "" H 10600 900 60  0000 C CNN
@@
 $EndComp
 $Comp
-L GND #PWR014
+L GND #PWR18
 U 1 1 53670BB1
 P 10600 2050
-F 0 "#PWR014" H 10600 2050 30  0001 C CNN
+F 0 "#PWR18" H 10600 2050 30  0001 C CNN
 F 1 "GND" H 10600 1980 30  0001 C CNN
 F 2 "" H 10600 2050 60  0000 C CNN
@@
 	10700 5750 10850 5750
 $Comp
-L +3.3V #PWR015
+L +3.3V #PWR19
 U 1 1 54575257
 P 10850 5750
-F 0 "#PWR015" H 10850 5710 30  0001 C CNN
+F 0 "#PWR19" H 10850 5710 30  0001 C CNN
 F 1 "+3.3V" H 10850 5860 30  0000 C CNN
 F 2 "" H 10850 5750 60  0000 C CNN
@@
 MCU5V
 $Comp
-L +5V #PWR016
+L +5V #PWR8
 U 1 1 5459D978
 P 5250 3700
-F 0 "#PWR016" H 5250 3790 20  0001 C CNN
+F 0 "#PWR8" H 5250 3790 20  0001 C CNN
 F 1 "+5V" H 5250 3790 30  0000 C CNN
 F 2 "~" H 5250 3700 60  0000 C CNN
@@
 WLED_N
 $Comp
-L +3.3V #PWR017
+L +3.3V #PWR14
 U 1 1 5465EE50
 P 7500 4000
-F 0 "#PWR017" H 7500 3960 30  0001 C CNN
+F 0 "#PWR14" H 7500 3960 30  0001 C CNN
 F 1 "+3.3V" H 7500 4110 30  0000 C CNN
 F 2 "" H 7500 4000 60  0000 C CNN
@@
 	4450 4850 4450 5100
 $Comp
-L GND #PWR018
+L GND #PWR6
 U 1 1 546D88C7
 P 4450 5100
-F 0 "#PWR018" H 4450 5100 30  0001 C CNN
+F 0 "#PWR6" H 4450 5100 30  0001 C CNN
 F 1 "GND" H 4450 5030 30  0001 C CNN
 F 2 "" H 4450 5100 60  0000 C CNN
@@
 $EndComp
 $Comp
-L +5V #PWR019
+L +5V #PWR12
 U 1 1 54752FD0
 P 6800 4000
-F 0 "#PWR019" H 6800 4090 20  0001 C CNN
+F 0 "#PWR12" H 6800 4090 20  0001 C CNN
 F 1 "+5V" H 6800 4090 30  0000 C CNN
 F 2 "~" H 6800 4000 60  0000 C CNN
@@
 Text Label 3050 2450 0    60   ~ 0
 LINK3
+$Comp
+L C_R_0603 R28
+U 1 1 5476A119
+P 5500 4400
+F 0 "R28" H 5550 4300 50  0000 C CNN
+F 1 "NO" H 5400 4300 50  0000 C CNN
+F 2 "C_R_0603" H 5500 4280 60  0001 C CNN
+F 3 "~" H 5500 4400 60  0000 C CNN
+	1    5500 4400
+	0    -1   -1   0
+$EndComp
+Wire Wire Line
+	5500 4600 5500 4800
+Connection ~ 5500 4800
+Wire Wire Line
+	5500 4200 5500 4050
+Wire Wire Line
+	5500 4050 5250 4050
+Connection ~ 5250 4050
 $EndSCHEMATC
