File: uPD720114.sch (KiCad schematic (older format))
At the start: 60 parts, among them U10 DLW21SN900SQ2, U13 IP4220CZ6, U14 IP4220CZ6, U15 AP2146, U16 AP2146, U2 DLW21SN900SQ2, U3 IP4220CZ6, U4 UPD720114-QFP48, U5 USB-AF-90, U9 DLW21SN900SQ2, X1 30MHz

Commit message: 整理到根目录
Parts:
- added JP9: IO_M02X1, IO_M02X1, symbol IO_M02X1
Connections:
- net at U4.28 (DM2): now also JP9.2
- net at U4.29 (DP2): now also JP9.1
Changed lines of the file:
@@
-EESchema Schematic File Version 2  date 2014/11/21 12:19:35
+EESchema Schematic File Version 2  date 2014/11/26 13:45:51
 LIBS:C
 LIBS:IC
@@
 Sheet 2 3
 Title ""
-Date "21 nov 2014"
+Date "26 nov 2014"
 Rev ""
 Comp ""
@@
 $EndComp
 $Comp
-L GND #PWR019
+L GND #PWR020
 U 1 1 534FC5F9
 P 2200 4150
-F 0 "#PWR019" H 2200 4050 30  0001 C CNN
+F 0 "#PWR020" H 2200 4050 30  0001 C CNN
 F 1 "GND" H 2200 4080 30  0001 C CNN
 F 2 "~" H 2200 4150 60  0000 C CNN
@@
 $EndComp
 $Comp
-L GND #PWR020
+L GND #PWR021
 U 1 1 534FCAE6
 P 3200 5250
-F 0 "#PWR020" H 3200 5150 30  0001 C CNN
+F 0 "#PWR021" H 3200 5150 30  0001 C CNN
 F 1 "GND" H 3200 5180 30  0001 C CNN
 F 2 "~" H 3200 5250 60  0000 C CNN
@@
 $EndComp
 $Comp
-L +3.3V #PWR021
+L +3.3V #PWR022
 U 1 1 534FCB20
 P 2150 4900
-F 0 "#PWR021" H 2150 5010 30  0001 C CNN
+F 0 "#PWR022" H 2150 5010 30  0001 C CNN
 F 1 "+3.3V" H 2150 5010 30  0000 C CNN
 F 2 "~" H 2150 4900 60  0000 C CNN
@@
 $EndComp
 $Comp
-L GND #PWR022
+L GND #PWR023
 U 1 1 534FCB5A
 P 4050 6550
-F 0 "#PWR022" H 4050 6450 30  0001 C CNN
+F 0 "#PWR023" H 4050 6450 30  0001 C CNN
 F 1 "GND" H 4050 6480 30  0001 C CNN
 F 2 "~" H 4050 6550 60  0000 C CNN
@@
 $EndComp
 $Comp
-L GND #PWR023
+L GND #PWR024
 U 1 1 534FD156
 P 1700 4950
-F 0 "#PWR023" H 1700 4850 30  0001 C CNN
+F 0 "#PWR024" H 1700 4850 30  0001 C CNN
 F 1 "GND" H 1700 4880 30  0001 C CNN
 F 2 "~" H 1700 4950 60  0000 C CNN
@@
 $EndComp
 $Comp
-L GND #PWR024
+L GND #PWR025
 U 1 1 534FD527
 P 2600 6250
-F 0 "#PWR024" H 2600 6150 30  0001 C CNN
+F 0 "#PWR025" H 2600 6150 30  0001 C CNN
 F 1 "GND" H 2600 6180 30  0001 C CNN
 F 2 "~" H 2600 6250 60  0000 C CNN
@@
 $EndComp
 $Comp
-L GND #PWR025
+L GND #PWR026
 U 1 1 534FD52D
 P 2800 6250
-F 0 "#PWR025" H 2800 6150 30  0001 C CNN
+F 0 "#PWR026" H 2800 6150 30  0001 C CNN
 F 1 "GND" H 2800 6180 30  0001 C CNN
 F 2 "~" H 2800 6250 60  0000 C CNN
@@
 $EndComp
 $Comp
-L GND #PWR026
+L GND #PWR027
 U 1 1 534FD533
 P 3000 6250
-F 0 "#PWR026" H 3000 6150 30  0001 C CNN
+F 0 "#PWR027" H 3000 6150 30  0001 C CNN
 F 1 "GND" H 3000 6180 30  0001 C CNN
 F 2 "~" H 3000 6250 60  0000 C CNN
@@
 $EndComp
 $Comp
-L GND #PWR027
+L GND #PWR028
 U 1 1 534FD71A
 P 2150 5750
-F 0 "#PWR027" H 2150 5650 30  0001 C CNN
+F 0 "#PWR028" H 2150 5650 30  0001 C CNN
 F 1 "GND" H 2150 5680 30  0001 C CNN
 F 2 "~" H 2150 5750 60  0000 C CNN
@@
 $EndComp
 $Comp
-L GND #PWR028
+L GND #PWR029
 U 1 1 534FDBB9
 P 1900 1450
-F 0 "#PWR028" H 1900 1350 30  0001 C CNN
+F 0 "#PWR029" H 1900 1350 30  0001 C CNN
 F 1 "GND" H 1900 1380 30  0001 C CNN
 F 2 "~" H 1900 1450 60  0000 C CNN
@@
 $EndComp
 $Comp
-L GND #PWR029
+L GND #PWR030
 U 1 1 534FDCFE
 P 2500 1700
-F 0 "#PWR029" H 2500 1600 30  0001 C CNN
+F 0 "#PWR030" H 2500 1600 30  0001 C CNN
 F 1 "GND" H 2500 1630 30  0001 C CNN
 F 2 "~" H 2500 1700 60  0000 C CNN
@@
 $EndComp
 $Comp
-L GND #PWR030
+L GND #PWR031
 U 1 1 535084C0
 P 2700 3150
-F 0 "#PWR030" H 2700 3050 30  0001 C CNN
+F 0 "#PWR031" H 2700 3050 30  0001 C CNN
 F 1 "GND" H 2700 3080 30  0001 C CNN
 F 2 "~" H 2700 3150 60  0000 C CNN
@@
 D+
 $Comp
-L GND #PWR031
+L GND #PWR032
 U 1 1 53508CE7
 P 3750 1550
-F 0 "#PWR031" H 3750 1450 30  0001 C CNN
+F 0 "#PWR032" H 3750 1450 30  0001 C CNN
 F 1 "GND" H 3750 1480 30  0001 C CNN
 F 2 "~" H 3750 1550 60  0000 C CNN
@@
 $EndComp
 $Comp
-L GND #PWR032
+L GND #PWR033
 U 1 1 53508CED
 P 4650 1550
-F 0 "#PWR032" H 4650 1450 30  0001 C CNN
+F 0 "#PWR033" H 4650 1450 30  0001 C CNN
 F 1 "GND" H 4650 1480 30  0001 C CNN
 F 2 "~" H 4650 1550 60  0000 C CNN
@@
 VBUS2
 $Comp
-L GND #PWR033
+L GND #PWR034
 U 1 1 53509F08
 P 8500 5750
-F 0 "#PWR033" H 8500 5650 30  0001 C CNN
+F 0 "#PWR034" H 8500 5650 30  0001 C CNN
 F 1 "GND" H 8500 5680 30  0001 C CNN
 F 2 "~" H 8500 5750 60  0000 C CNN
@@
 $EndComp
 $Comp
-L GND #PWR034
+L GND #PWR035
 U 1 1 5350A075
 P 9000 5650
-F 0 "#PWR034" H 9000 5550 30  0001 C CNN
+F 0 "#PWR035" H 9000 5550 30  0001 C CNN
 F 1 "GND" H 9000 5580 30  0001 C CNN
 F 2 "~" H 9000 5650 60  0000 C CNN
@@
 $EndComp
 $Comp
-L GND #PWR035
+L GND #PWR036
 U 1 1 5350A07B
 P 9400 5650
-F 0 "#PWR035" H 9400 5550 30  0001 C CNN
+F 0 "#PWR036" H 9400 5550 30  0001 C CNN
 F 1 "GND" H 9400 5580 30  0001 C CNN
 F 2 "~" H 9400 5650 60  0000 C CNN
@@
 $EndComp
 $Comp
-L GND #PWR036
+L GND #PWR037
 U 1 1 5350A582
 P 8600 6700
-F 0 "#PWR036" H 8600 6600 30  0001 C CNN
+F 0 "#PWR037" H 8600 6600 30  0001 C CNN
 F 1 "GND" H 8600 6630 30  0001 C CNN
 F 2 "~" H 8600 6700 60  0000 C CNN
@@
 $EndComp
 $Comp
-L GND #PWR037
+L GND #PWR038
 U 1 1 5350A588
 P 9000 6700
-F 0 "#PWR037" H 9000 6600 30  0001 C CNN
+F 0 "#PWR038" H 9000 6600 30  0001 C CNN
 F 1 "GND" H 9000 6630 30  0001 C CNN
 F 2 "~" H 9000 6700 60  0000 C CNN
@@
 $EndComp
 $Comp
-L GND #PWR038
+L GND #PWR039
 U 1 1 5350A58E
 P 9400 6700
-F 0 "#PWR038" H 9400 6600 30  0001 C CNN
+F 0 "#PWR039" H 9400 6600 30  0001 C CNN
 F 1 "GND" H 9400 6630 30  0001 C CNN
 F 2 "~" H 9400 6700 60  0000 C CNN
@@
 VBUS4
 $Comp
-L GND #PWR039
+L GND #PWR040
 U 1 1 5350AC40
 P 5350 4850
-F 0 "#PWR039" H 5350 4750 30  0001 C CNN
+F 0 "#PWR040" H 5350 4750 30  0001 C CNN
 F 1 "GND" H 5350 4780 30  0001 C CNN
 F 2 "~" H 5350 4850 60  0000 C CNN
@@
 $EndComp
 $Comp
-L GND #PWR040
+L GND #PWR041
 U 1 1 5350BC51
 P 8400 4400
-F 0 "#PWR040" H 8400 4300 30  0001 C CNN
+F 0 "#PWR041" H 8400 4300 30  0001 C CNN
 F 1 "GND" H 8400 4330 30  0001 C CNN
 F 2 "~" H 8400 4400 60  0000 C CNN
@@
 $EndComp
 $Comp
-L GND #PWR041
+L GND #PWR042
 U 1 1 5350BFE2
 P 7200 4400
-F 0 "#PWR041" H 7200 4300 30  0001 C CNN
+F 0 "#PWR042" H 7200 4300 30  0001 C CNN
 F 1 "GND" H 7200 4330 30  0001 C CNN
 F 2 "~" H 7200 4400 60  0000 C CNN
@@
 $EndComp
 $Comp
-L GND #PWR042
+L GND #PWR043
 U 1 1 5350CD4A
 P 10850 3450
-F 0 "#PWR042" H 10850 3350 30  0001 C CNN
+F 0 "#PWR043" H 10850 3350 30  0001 C CNN
 F 1 "GND" H 10850 3380 30  0001 C CNN
 F 2 "~" H 10850 3450 60  0000 C CNN
@@
 $EndComp
 $Comp
-L GND #PWR043
+L GND #PWR044
 U 1 1 5350D046
 P 7200 3500
-F 0 "#PWR043" H 7200 3400 30  0001 C CNN
+F 0 "#PWR044" H 7200 3400 30  0001 C CNN
 F 1 "GND" H 7200 3430 30  0001 C CNN
 F 2 "~" H 7200 3500 60  0000 C CNN
@@
 $EndComp
 $Comp
-L GND #PWR044
+L GND #PWR045
 U 1 1 5350D04C
 P 8400 3500
-F 0 "#PWR044" H 8400 3400 30  0001 C CNN
+F 0 "#PWR045" H 8400 3400 30  0001 C CNN
 F 1 "GND" H 8400 3430 30  0001 C CNN
 F 2 "~" H 8400 3500 60  0000 C CNN
@@
 	10150 3300 10250 3300
 $Comp
-L +5V #PWR045
+L +5V #PWR046
 U 1 1 545AE01A
 P 1900 800
-F 0 "#PWR045" H 1900 890 20  0001 C CNN
+F 0 "#PWR046" H 1900 890 20  0001 C CNN
 F 1 "+5V" H 1900 890 30  0000 C CNN
 F 2 "~" H 1900 800 60  0000 C CNN
@@
 $EndComp
 $Comp
-L +5V #PWR046
+L +5V #PWR047
 U 1 1 545AE027
 P 1100 2950
-F 0 "#PWR046" H 1100 3040 20  0001 C CNN
+F 0 "#PWR047" H 1100 3040 20  0001 C CNN
 F 1 "+5V" H 1100 3040 30  0000 C CNN
 F 2 "~" H 1100 2950 60  0000 C CNN
@@
 $EndComp
 $Comp
-L +5V #PWR047
+L +5V #PWR048
 U 1 1 545AE02D
 P 8500 4850
-F 0 "#PWR047" H 8500 4940 20  0001 C CNN
+F 0 "#PWR048" H 8500 4940 20  0001 C CNN
 F 1 "+5V" H 8500 4940 30  0000 C CNN
 F 2 "~" H 8500 4850 60  0000 C CNN
@@
 $EndComp
 $Comp
-L +5V #PWR048
+L +5V #PWR049
 U 1 1 545AE033
 P 8600 6000
-F 0 "#PWR048" H 8600 6090 20  0001 C CNN
+F 0 "#PWR049" H 8600 6090 20  0001 C CNN
 F 1 "+5V" H 8600 6090 30  0000 C CNN
 F 2 "~" H 8600 6000 60  0000 C CNN
@@
 	1    0    0    -1
 $EndComp
+$Comp
+L IO_M02X1 JP9
+U 1 1 54741E5A
+P 5500 3050
+F 0 "JP9" H 5480 2860 60  0000 C CNN
+F 1 "IO_M02X1" H 5490 3240 60  0000 C CNN
+F 2 "IO_M02X1" H 5490 3240 60  0001 C CNN
+F 3 "~" H 5500 3050 60  0000 C CNN
+	1    5500 3050
+	-1   0    0    1
+$EndComp
+Wire Wire Line
+	5200 3000 5250 3000
+Wire Wire Line
+	5200 3100 5250 3100
 $EndSCHEMATC
