File: Vocore/ATMEGA32U4.sch (KiCad schematic (older format))
At the start: 20 parts, among them IC1 IC_ATMEGA32U4_TQFP44, X2 16m

Commit message: Vocore第二版修改完成
Parts:
- removed JP4: IO_M08X2, IO_M08X2, symbol IO_M08X2
- added JP6: IO_M07X2, IO_M07X2, symbol IO_M07X2
Connections:
- net +5V: no longer JP7.15
- net D0/RX: now also JP6.1
- net D1/TX: now also JP6.2
- net D2/SDA: now also JP6.3
- net D3/SCL: now also JP6.4
- net D4: now also JP6.5
- net D5*: now also JP6.6
- net D6*: now also JP6.7
- net D7: now also JP6.8
- net GND: now also JP7.15
- net IO10*: now also JP6.11
- net IO11*: now also JP6.12
- net IO12: now also JP6.13
- net IO13*: now also JP6.14
- net IO8: now also JP6.9
- net IO9*: now also JP6.10
Changed lines of the file:
@@
-EESchema Schematic File Version 2  date 2014/12/30 17:54:50
+EESchema Schematic File Version 2  date 2015/1/14 16:22:56
 LIBS:C
 LIBS:IC
@@
 LIBS:rcl
 LIBS:gl
+LIBS:ATMEGA32U4-cache
+LIBS:uPD720114-cache
+LIBS:vc-cache
+LIBS:vocore-cache
+LIBS:SchumyHao
 LIBS:vocore-cache
 EELAYER 27 0
@@
 Sheet 3 3
 Title ""
-Date "30 dec 2014"
+Date "14 jan 2015"
 Rev ""
 Comp ""
@@
 Text Label 10400 6200 0    60   ~ 0
 GND
-Text Label 9000 4600 2    60   ~ 0
-+5V
-Text Label 10400 4600 0    60   ~ 0
-GND
 Text Label 10400 6300 0    60   ~ 0
 +3.3V
-Text Label 9000 6400 2    60   ~ 0
-+5V
 Text Label 10400 6400 0    60   ~ 0
 GND
-$Comp
-L IO_M08X2 JP4
-U 1 1 549BB08F
-P 9650 4700
-F 0 "JP4" H 9680 5045 60  0000 C CNN
-F 1 "IO_M08X2" H 9700 4950 60  0000 C CNN
-F 2 "IO_M08X2" H 9700 3960 60  0001 C CNN
-F 3 "~" H 9650 4700 60  0000 C CNN
-	1    9650 4700
-	1    0    0    -1
-$EndComp
 $Comp
 L IO_M08X2 JP7
@@
 $EndComp
 Wire Wire Line
-	10150 4600 10400 4600
-Wire Wire Line
 	10150 4700 10400 4700
 Wire Wire Line
@@
 	10150 5300 10400 5300
 Wire Wire Line
-	9250 4600 9000 4600
-Wire Wire Line
 	9250 4700 9000 4700
 Wire Wire Line
@@
 Wire Wire Line
 	10400 6400 10150 6400
+$Comp
+L IO_M07X2 JP6
+U 1 1 54B499D6
+P 9650 4800
+F 0 "JP6" H 9680 5145 60  0000 C CNN
+F 1 "IO_M07X2" H 9700 5050 60  0000 C CNN
+F 2 "IO_M07X2" H 9700 4170 60  0001 C CNN
+F 3 "~" H 9650 4800 60  0000 C CNN
+	1    9650 4800
+	1    0    0    -1
+$EndComp
+Text Label 9000 6400 2    60   ~ 0
+GND
 $EndSCHEMATC
