File: Vocore/vocore.sch (KiCad schematic (older format))
At the start: 40 parts, among them J1 IO_USB-MICRO-B-MK5P, P2 IO_HOLE-3.2, P3 IO_HOLE-3.2, U1 IC_MP1484EN_SOIC08, U11 C_SW_SPSDSMD, U17 C_SW_SPSDSMD, U8 FT232RL_SSOP_28

Commit message: Vocore第二版修改完成
Parts:
- removed JP5, JP6: IO_M08X2, IO_M08X2, symbol IO_M08X2
- removed S1: C_SW_TS42, C_SW_TS42, symbol C_SW_TS42
- added C48: 104, C_C_0603, symbol C_C_0603
- added JP4: IO_M06X2, IO_M06X2, symbol IO_M06X2
- added JP5: IO_M07X2, IO_M07X2, symbol IO_M07X2
- added R28: 200, C_R_0603, symbol C_R_0603
- added S1: C_SW_1505, C_SW_1505, symbol C_SW_1505
Connections:
- wire segments 212 -> 206

Commit message: modify  PCB
Parts:
- removed JP3: IO_M19X1, IO-M19X1-1.27MM, symbol IO_M19X1
- added JP10: IO_M18X1, IO-M18X1-1.27MM, symbol IO_M18X1
Connections:
- net G#03/SPI_CS0: now also JP10.13
- net G#06/SPI_MISO: now also JP10.14
- net G#07/I2S_CLK: now also JP10.17
- net G#10/I2S_SDI/RXD: now also JP10.15
- net G#11/PCM_FS: now also JP10.12
- net G#15/TXD2: now also JP10.18
- net G#16/RXD2: now also JP10.16
- net P0RN: now also JP10.8
- net P0RP: now also JP10.9
- net P0TN: now also JP10.11
- net P0TP: now also JP10.10
- net P4RN: now also JP10.4
- net P4RP: now also JP10.5
- net P4TN: now also JP10.7
- net P4TP: now also JP10.6
- net USB+: now also JP10.2
- net USB-: now also JP10.3
Changed lines of the file:
@@
-EESchema Schematic File Version 2  date 2015/1/14 16:22:56
+EESchema Schematic File Version 2
 LIBS:C
 LIBS:IC
@@
 LIBS:power
 LIBS:rcl
-LIBS:gl
 LIBS:ATMEGA32U4-cache
 LIBS:uPD720114-cache
 LIBS:vc-cache
 LIBS:vocore-cache
-LIBS:SchumyHao
 LIBS:vocore-cache
 EELAYER 27 0
@@
 Sheet 1 3
 Title ""
-Date "14 jan 2015"
+Date "10 mar 2015"
 Rev ""
 Comp ""
@@
 Text Label 1550 5650 2    60   ~ 0
 G#15/TXD2
-Text Label 1550 5750 2    60   ~ 0
-GND
 Text Label 10850 6250 0    60   ~ 0
 USB+
@@
 Text Label 8650 4450 0    60   ~ 0
 RD-
-$Comp
-L IO_M19X1 JP3
-U 1 1 54991128
-P 1900 4850
-F 0 "JP3" H 1755 5895 60  0000 C CNN
-F 1 "IO_M19X1" H 1805 5800 60  0000 C CNN
-F 2 "IO-M19X1-1.27MM" H 1815 3800 60  0001 C CNN
-F 3 "~" H 1900 4950 60  0000 C CNN
-	1    1900 4850
-	-1   0    0    -1
-$EndComp
 $Comp
 L C_SW_SPSDSMD U17
@@
 	1550 5650 1800 5650
 Wire Wire Line
-	1550 5750 1800 5750
-Wire Wire Line
 	1800 1250 1550 1250
 Wire Wire Line
@@
 Wire Wire Line
 	8200 6100 8650 6100
-Wire Wire Line
-	1800 4250 1550 4250
-Wire Wire Line
-	1800 4150 1550 4150
-Wire Wire Line
-	1800 4050 1550 4050
 Wire Wire Line
 	8450 5000 8650 5000
@@
 Text Label 2750 7550 2    60   ~ 0
 GND
+$Comp
+L IO_M18X1 JP10
+U 1 1 54FE574D
+P 1900 4750
+F 0 "JP10" H 1755 5795 60  0000 C CNN
+F 1 "IO_M18X1" H 1805 5700 60  0000 C CNN
+F 2 "IO-M18X1-1.27MM" H 1815 3700 60  0001 C CNN
+F 3 "~" H 1900 4750 60  0000 C CNN
+	1    1900 4750
+	-1   0    0    -1
+$EndComp
+Wire Wire Line
+	1550 4050 1800 4050
+Wire Wire Line
+	1550 4150 1800 4150
+Wire Wire Line
+	1550 4250 1800 4250
 $EndSCHEMATC
